Commit message: Tweaks and comments

File: src/sphero_rvr_description/urdf/sphero_rvr.urdf.xacro (robot description, xacro)
@@ -1,5 +1,5 @@
 <?xml version="1.0"?>
 <robot xmlns:xacro="http://www.ros.org/wiki/xacro" name="track_robot">
-    <!--common-->
+    <!-- common -->
     <xacro:include filename="$(find sphero_rvr_description)/urdf/common.urdf.xacro" />
     <xacro:include filename="$(find sphero_rvr_description)/urdf/materials.urdf.xacro" />
@@ -10,8 +10,9 @@
     <!-- urg laser -->
     <xacro:include filename="$(find urg_node)/urdf/hokuyo_ust10.urdf.xacro" />
-    <!-- dummy base link no inertia to satisfy kdl -->
+    <!-- base_footprint is on the ground under the robot -->
+    <link name="base_footprint"/>
+    <!-- dummy base_link no inertia to satisfy kdl -->
     <link name="base_link"/>
-    <!-- Base footprint is on the ground under the robot -->
-    <link name="base_footprint"/>
+    <!-- attach base_link to base_footprint -->
     <joint name="base_footprint_joint" type="fixed">
         <origin xyz="0 0 ${rvr_track_dz - rvr_wheel_radius}" rpy="0 0 0" />
@@ -43,5 +44,4 @@
         <origin xyz="${-0.03} 0 ${rvr_body_height + 0.035}" rpy="0 0 0" />
     </xacro:hokuyo_ust10_mount>
-    <!-- gazebo extras -->
     <!-- gazebo control -->
     <gazebo>

Commit message: Try to fix disconnected tf tree

File: src/sphero_rvr_description/urdf/sphero_rvr.urdf.xacro (robot description, xacro)
@@ -12,11 +12,11 @@
     <!-- base_footprint is on the ground under the robot -->
     <link name="base_footprint"/>
-    <!-- dummy base_link no inertia to satisfy kdl -->
+    <!-- base_link is on the rvr -->
     <link name="base_link"/>
     <!-- attach base_link to base_footprint -->
     <joint name="base_footprint_joint" type="fixed">
         <origin xyz="0 0 ${rvr_track_dz - rvr_wheel_radius}" rpy="0 0 0" />
-        <parent link="base_link" />
-        <child link="base_footprint" />
+        <parent link="base_footprint" />
+        <child link="base_link" />
     </joint>
     <!-- attach body to base_link -->
